File: assets/ESP32+TIPS122 Version 2/ESP32+TIPS/ESP32+TIPS (1).kicad_pcb (KiCad board)
At the start: 2 copper layers, 88 parts, among them J1 Conn_01x03_Pin, J2 DB25_Socket, J3 Screw_Terminal_01x02, Q1 TIP122, Q10 TIP122, Q11 TIP122, Q12 TIP122, Q13 TIP122, Q14 TIP122, Q15 TIP122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

Commit message: update pcb
Parts:
- moved .1 2.55 mm to (169.5, 164.2)
- moved .10 2.55 mm to (169.0, 37.8)
- moved .11 2.55 mm to (259.5, 159.8)
- moved .12 2.55 mm to (259.5, 144.8)
- moved .13 2.55 mm to (259.5, 129.8)
- moved .14 2.55 mm to (259.5, 116.2)
- moved .15 2.55 mm to (259.5, 102.2)
- moved .16 2.55 mm to (259.5, 88.8)
- moved .17 2.55 mm to (259.5, 74.8)
- moved .18 2.55 mm to (259.5, 60.8)
- moved .19 2.55 mm to (259.5, 46.8)
- moved .2 2.55 mm to (169.5, 150.2)
- moved .20 2.55 mm to (259.5, 33.2)
- moved .3 2.55 mm to (169.5, 136.2)
- moved .4 2.55 mm to (169.5, 122.8)
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Routing:
- net Net-(U2-D14): track 249.0 -> 270.9 mm
- net Net-(U2-D12): track 289.7 -> 307.2 mm
- net VCC: track 239.4 -> 255.9 mm
- net Net-(U2-D13): track 264.1 -> 275.6 mm
- net Net-(U2-D32): track 108.2 -> 117.3 mm
- net Net-(U2-TX2): track 178.1 -> 186.0 mm
- net Net-(U2-D22): track 109.4 -> 115.5 mm
- net Net-(U2-RX2): track 151.7 -> 157.4 mm
- net Net-(Q11-C): track 590.9 -> 596.5 mm
- net GND: track 972.3 -> 977.6 mm
- net Net-(U2-D33): track 132.9 -> 136.8 mm
- net Net-(U2-D27): track 74.2 -> 77.6 mm
- net Net-(J2-P19): track 131.8 -> 134.2 mm
- net Net-(U2-D21): track 249.7 -> 251.6 mm
- net Net-(U2-D34): track 164.5 -> 166.3 mm
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